Commit message: change

File: gui/urdf/body.xacro (robot description, xacro)
@@ -5,5 +5,8 @@
     </material>
     <material name="red">
-        <color rgba="1.0 0.0 0.0 2.5"/>
+        <color rgba="1.0 0.0 0.0 2.0"/>
+    </material>
+    <material name="white">
+        <color rgba="0.5 0.0 2.5 2.0"/>
     </material>
     <xacro:macro name="flipper_macro" params="parent suffix xyz">
@@ -20,5 +23,5 @@
                 </geometry>
                 <origin xyz="0 0 0.055" rpy="0 0 0"/>
-                <material name="gray"/>
+                <material name="red"/>
             </visual>
         </link>
@@ -36,5 +39,5 @@
                 <box size="0.34 0.15 0.06"/>
             </geometry>
-            <material name="gray"/>
+            <material name="white"/>
         </visual>
     </link>
